File: Environment_Sensor_PCBs/hpma115c0-004_adapter.sch (EAGLE design)
At the start: 10 parts, among them U1 BME680

Commit message: Adding most recent boards
Parts:
- removed C1, C2: 100nF, daneagle_db8.0:CAP_NP_0402
- removed C3: 10uF, daneagle_db8.0:CAP_POL_SMD_1206
- removed IN, OUT: 53261-04, con-molex:53261-04
- removed R0X76: 0r, daneagle_db8.0:RESISTOR_0402
- removed R0X77: dnp, daneagle_db8.0:RESISTOR_0402
- removed R1, R2: 4k7, daneagle_db8.0:RESISTOR_0402
- removed U1: BME680, daneagle_db8.0:BME680_GAS_AQ/BARO/TEMP/HUMID-I2C-SPI
- added CON1: HEADER_5X2_SFM-105-02-H-D, daneagle_db8.0:HEADER_5X2_SFM-105-02-H-D
- added RTX, RX, TRX, TX: DNP, daneagle_db8.0:RESISTOR_0402
- added X1: 53261-04, con-molex:53261-04
Connections:
- removed net 3V3: C1.P$1, C2.P$1, C3.P, IN-1.S, OUT-1.S, R0X77.P$1, R1.P$2, R2.P$2, U1.CSB, U1.VCC, U1.VCCIO
- removed net ADDR: R0X76.P$2, R0X77.P$2, U1.SDO/ADR
- removed net SCL: IN-4.S, OUT-4.S, R2.P$1, U1.SCK/SCL
- removed net SDA: IN-2.S, OUT-2.S, R1.P$1, U1.SDI/SDA
- new net RX: CON1.P$7, RTX.P$2, RX.P$1, RX.P$2, TX.P$1, X1-2.S
- new net TX: CON1.P$9, RTX.P$1, TRX.P$1, TRX.P$2, TX.P$2, X1-4.S
- new net VCC: CON1.P$2, X1-1.S
- net GND: now also CON1.P$3, CON1.P$4, X1-3.S; no longer C1.P$2, C2.P$2, C3.N, IN-3.S, OUT-3.S, R0X76.P$1, U1.GND
Other:
- note removed: "DNP unless not present on control board"
